Commit message: Implement C++ GoalStopManager node and optimize Gazebo wheel joint damping, friction, and PID gains to prevent vehicle drift

File: autocar_description/urdf/car.xacro (robot description, xacro)
@@ -166,5 +166,5 @@
     <axis xyz="0 0 1"/>
     <limit lower="-0.785" upper="0.785" effort="80.0" velocity="4.0"/>
-    <dynamics damping="0.5" friction="0.1"/>
+    <dynamics damping="3.0" friction="0.8"/>
   </joint>
   <!-- Front Right Steering Knuckle -->
@@ -189,5 +189,5 @@
     <axis xyz="0 0 1"/>
     <limit lower="-0.785" upper="0.785" effort="80.0" velocity="4.0"/>
-    <dynamics damping="0.5" friction="0.1"/>
+    <dynamics damping="3.0" friction="0.8"/>
   </joint>
   <!-- ===================== -->
@@ -299,5 +299,5 @@
     <axis xyz="0 1 0"/>
     <limit effort="100.0" velocity="15.0"/>
-    <dynamics damping="0.1" friction="0.1"/>
+    <dynamics damping="1.5" friction="0.5"/>
   </joint>
   <!-- Front Right Wheel (attached to steering knuckle) -->
@@ -308,5 +308,5 @@
     <axis xyz="0 1 0"/>
     <limit effort="100.0" velocity="15.0"/>
-    <dynamics damping="0.1" friction="0.1"/>
+    <dynamics damping="1.5" friction="0.5"/>
   </joint>
   <!-- Rear Left Wheel (fixed steering, connected to base_link) -->
@@ -317,5 +317,5 @@
     <axis xyz="0 1 0"/>
     <limit effort="100.0" velocity="15.0"/>
-    <dynamics damping="0.1" friction="0.1"/>
+    <dynamics damping="1.5" friction="0.5"/>
   </joint>
   <!-- Rear Right Wheel (fixed steering, connected to base_link) -->
@@ -326,5 +326,5 @@
     <axis xyz="0 1 0"/>
     <limit effort="100.0" velocity="15.0"/>
-    <dynamics damping="0.1" friction="0.1"/>
+    <dynamics damping="1.5" friction="0.5"/>
   </joint>
   <!-- ===================== -->
